File: arduino-nano-breakout-1/arduino-nano-breakout-1/arduino-nano-breakout-1.kicad_pcb (KiCad board)
At the start: 4 copper layers, 7 x 7 mm, 4 parts, among them J1 PJ-002A, J2 Conn_01x03_Male, J4 Conn_01x08_Male

Commit message: power lines
Parts:
- moved J2 5.08 mm to (149.9, 110.5), turned to 0 degrees
Routing:
- net Net-(A1-Pad30): track 121.4 -> 52.1 mm, vias 0 -> 2
- net GND: track 32.2 -> 65.4 mm, vias 2 -> 1
- net Net-(A1-Pad27): track 59.0 -> 42.7 mm, vias 0 -> 2
- net Net-(J1-Pad1): track 13.8 -> 14.5 mm
Other:
- copper layers 4 -> 2
Changed lines of the file:
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@@
     (thickness 1.6)
     (drawings 0)
-    (tracks 74)
+    (tracks 65)
     (zones 0)
     (modules 4)
@@
   (layers
     (0 F.Cu signal)
-    (1 In1.Cu signal)
-    (2 In2.Cu signal)
     (31 B.Cu signal)
     (32 B.Adhes user)
@@
     (solder_mask_min_width 0.25)
     (aux_axis_origin 0 0)
-    (visible_elements FFFFFF7F)
+    (visible_elements 7FFFFFFF)
     (pcbplotparams
       (layerselection 0x010fc_ffffffff)
@@
   )
   (module Connector_PinHeader_2.54mm:PinHeader_1x03_P2.54mm_Vertical (layer F.Cu)
-    (at 149.86 115.57 180)
+    (at 149.86 110.49)
     (descr "Through hole straight pin header, 1x03, 2.54mm pitch, single row")
     (tags "Through hole pin header THT 1x03 2.54mm single row")
-    (fp_text reference J2 (at 0 -2.33 180) (layer F.SilkS)
-      (effects (font (size 1 1) (thickness 0.15)))
-    )
-    (fp_text value Conn_01x03_Male (at 0 7.41 180) (layer F.Fab)
+    (fp_text reference J2 (at 0 -2.33) (layer F.SilkS)
+      (effects (font (size 1 1) (thickness 0.15)))
+    )
+    (fp_text value Conn_01x03_Male (at 0 7.41) (layer F.Fab)
       (effects (font (size 1 1) (thickness 0.15)))
     )
@@
     (fp_line (start 1.8 6.85) (end 1.8 -1.8) (layer F.CrtYd) (width 0.05))
     (fp_line (start 1.8 -1.8) (end -1.8 -1.8) (layer F.CrtYd) (width 0.05))
-    (fp_text user %R (at 0 2.54 270) (layer F.Fab)
-      (effects (font (size 1 1) (thickness 0.15)))
-    )
-    (pad 1 thru_hole rect (at 0 0 180) (size 1.7 1.7) (drill 1) (layers *.Cu *.Mask)
+    (fp_text user %R (at 0 2.54 90) (layer F.Fab)
+      (effects (font (size 1 1) (thickness 0.15)))
+    )
+    (pad 1 thru_hole rect (at 0 0) (size 1.7 1.7) (drill 1) (layers *.Cu *.Mask)
       (net 18 "Net-(A1-Pad27)"))
-    (pad 2 thru_hole oval (at 0 2.54 180) (size 1.7 1.7) (drill 1) (layers *.Cu *.Mask)
+    (pad 2 thru_hole oval (at 0 2.54) (size 1.7 1.7) (drill 1) (layers *.Cu *.Mask)
       (net 24 "Net-(J1-Pad1)"))
-    (pad 3 thru_hole oval (at 0 5.08 180) (size 1.7 1.7) (drill 1) (layers *.Cu *.Mask)
+    (pad 3 thru_hole oval (at 0 5.08) (size 1.7 1.7) (drill 1) (layers *.Cu *.Mask)
       (net 21 "Net-(A1-Pad30)"))
     (model ${KISYS3DMOD}/Connector_PinHeader_2.54mm.3dshapes/PinHeader_1x03_P2.54mm_Vertical.wrl
@@
     )
   )
-  (via (at 157.48 113.03) (size 1.6) (drill 0.4) (layers F.Cu B.Cu) (net 7))
   (segment (start 134.62 78.74) (end 129.54 83.82) (width 0.25) (layer F.Cu) (net 7))
   (segment (start 144.78 78.74) (end 134.62 78.74) (width 0.25) (layer F.Cu) (net 7))
-  (segment (start 144.78 78.74) (end 146.05 78.74) (width 0.25) (layer F.Cu) (net 7))
-  (segment (start 147.32 77.47) (end 152.4 77.47) (width 0.25) (layer F.Cu) (net 7))
-  (segment (start 146.05 78.74) (end 147.32 77.47) (width 0.25) (layer F.Cu) (net 7))
-  (segment (start 157.48 110.14) (end 157.48 111.904999) (width 1.4) (layer F.Cu) (net 7))
-  (segment (start 157.48 111.904999) (end 157.48 113.03) (width 1.4) (layer F.Cu) (net 7))
-  (segment (start 152.4 77.47) (end 156.21 77.47) (width 1.4) (layer F.Cu) (net 7))
+  (segment (start 144.78 78.74) (end 146.05 78.74) (width 1.6) (layer F.Cu) (net 7))
+  (segment (start 147.32 77.47) (end 152.4 77.47) (width 1.6) (layer F.Cu) (net 7))
+  (segment (start 146.05 78.74) (end 147.32 77.47) (width 1.6) (layer F.Cu) (net 7))
+  (segment (start 152.4 77.47) (end 156.21 77.47) (width 2.4) (layer F.Cu) (net 7))
   (via (at 152.4 77.47) (size 1.6) (drill 0.4) (layers F.Cu B.Cu) (net 7))
-  (segment (start 148.59 80.01) (end 144.78 83.82) (width 0.25) (layer F.Cu) (net 18))
-  (segment (start 156.21 80.01) (end 148.59 80.01) (width 0.25) (layer F.Cu) (net 18))
-  (segment (start 147.61 115.57) (end 149.86 115.57) (width 1.4) (layer F.Cu) (net 18))
-  (segment (start 147.32 115.28) (end 147.61 115.57) (width 1.4) (layer F.Cu) (net 18))
-  (segment (start 156.21 80.01) (end 157.48 80.01) (width 1.4) (layer F.Cu) (net 18))
-  (segment (start 157.48 80.01) (end 158.75 81.28) (width 1.4) (layer F.Cu) (net 18))
-  (segment (start 158.75 81.28) (end 158.75 99.06) (width 1.4) (layer F.Cu) (net 18))
-  (segment (start 158.75 99.06) (end 157.48 100.33) (width 1.4) (layer F.Cu) (net 18))
-  (segment (start 157.48 100.33) (end 154.94 100.33) (width 1.4) (layer F.Cu) (net 18))
-  (segment (start 147.32 107.95) (end 147.32 115.28) (width 1.4) (layer F.Cu) (net 18))
-  (segment (start 154.94 100.33) (end 147.32 107.95) (width 1.4) (layer F.Cu) (net 18))
-  (segment (start 142.24 73.66) (end 144.78 76.2) (width 0.25) (layer F.Cu) (net 21))
-  (segment (start 161.29 104.14) (end 160.02 105.41) (width 0.25) (layer F.Cu) (net 21))
-  (segment (start 128.27 73.66) (end 142.24 73.66) (width 0.25) (layer F.Cu) (net 21))
-  (segment (start 153.67 109.22) (end 153.67 115.57) (width 0.25) (layer F.Cu) (net 21))
-  (segment (start 161.29 102.87) (end 161.29 104.14) (width 0.25) (layer F.Cu) (net 21))
-  (segment (start 160.02 101.6) (end 161.29 102.87) (width 0.25) (layer F.Cu) (net 21))
-  (segment (start 156.21 101.6) (end 160.02 101.6) (width 0.25) (layer F.Cu) (net 21))
-  (segment (start 149.86 110.49) (end 149.86 107.95) (width 0.25) (layer F.Cu) (net 21))
-  (segment (start 130.81 116.84) (end 127 113.03) (width 0.25) (layer F.Cu) (net 21))
-  (segment (start 149.86 107.95) (end 156.21 101.6) (width 0.25) (layer F.Cu) (net 21))
-  (segment (start 160.02 106.68) (end 158.75 107.95) (width 0.25) (layer F.Cu) (net 21))
-  (segment (start 160.02 105.41) (end 160.02 106.68) (width 0.25) (layer F.Cu) (net 21))
-  (segment (start 158.75 107.95) (end 154.94 107.95) (width 0.25) (layer F.Cu) (net 21))
-  (segment (start 154.94 107.95) (end 153.67 109.22) (width 0.25) (layer F.Cu) (net 21))
-  (segment (start 153.67 115.57) (end 152.4 116.84) (width 0.25) (layer F.Cu) (net 21))
-  (segment (start 152.4 116.84) (end 130.81 116.84) (width 0.25) (layer F.Cu) (net 21))
-  (segment (start 127 113.03) (end 127 74.93) (width 0.25) (layer F.Cu) (net 21))
-  (segment (start 127 74.93) (end 128.27 73.66) (width 0.25) (layer F.Cu) (net 21))
+  (segment (start 152.4 77.47) (end 152.4 81.28) (width 2.4) (layer B.Cu) (net 7))
+  (segment (start 152.4 81.28) (end 152.4 106.68) (width 2.4) (layer B.Cu) (net 7))
+  (segment (start 152.895 106.68) (end 156.355 110.14) (width 2.4) (layer B.Cu) (net 7))
+  (segment (start 152.4 106.68) (end 152.895 106.68) (width 0.25) (layer B.Cu) (net 7))
+  (segment (start 157.48 110.49) (end 157.48 110.14) (width 0.25) (layer F.Cu) (net 7))
+  (segment (start 157.48 110.14) (end 156.355 110.14) (width 2.4) (layer B.Cu) (net 7))
+  (segment (start 149.86 110.49) (end 148.59 109.22) (width 2.4) (layer F.Cu) (net 18))
+  (segment (start 148.59 109.22) (end 148.59 106.68) (width 2.4) (layer F.Cu) (net 18))
+  (via (at 148.59 81.28) (size 1.6) (drill 0.4) (layers F.Cu B.Cu) (net 18))
+  (segment (start 148.59 106.68) (end 148.59 106.68) (width 2.4) (layer F.Cu) (net 18))
+  (via (at 148.59 106.68) (size 1.6) (drill 0.4) (layers F.Cu B.Cu) (net 18))
+  (segment (start 149.86 80.01) (end 148.59 81.28) (width 2.4) (layer F.Cu) (net 18))
+  (segment (start 156.21 80.01) (end 149.86 80.01) (width 2.4) (layer F.Cu) (net 18))
+  (segment (start 146.05 83.82) (end 144.78 83.82) (width 1.6) (layer F.Cu) (net 18))
+  (segment (start 148.59 81.28) (end 146.05 83.82) (width 1.6) (layer F.Cu) (net 18))
+  (segment (start 148.59 81.28) (end 148.59 106.68) (width 2.4) (layer B.Cu) (net 18))
+  (segment (start 149.86 115.57) (end 140.97 115.57) (width 1.6) (layer F.Cu) (net 21))
+  (segment (start 140.97 115.57) (end 140.97 115.57) (width 1.6) (layer F.Cu) (net 21))
+  (via (at 140.97 115.57) (size 1.6) (drill 0.4) (layers F.Cu B.Cu) (net 21))
+  (segment (start 140.97 115.57) (end 140.97 76.2) (width 1.6) (layer B.Cu) (net 21))
+  (segment (start 140.97 76.2) (end 140.97 76.2) (width 1.6) (layer B.Cu) (net 21))
+  (via (at 140.97 76.2) (size 1.6) (drill 0.4) (layers F.Cu B.Cu) (net 21))
+  (segment (start 140.97 76.2) (end 144.78 76.2) (width 1.6) (layer F.Cu) (net 21))
   (segment (start 150.09 113.03) (end 149.86 113.03) (width 0.25) (layer F.Cu) (net 24))
-  (segment (start 149.86 113.03) (end 151.13 113.03) (width 1.4) (layer F.Cu) (net 24))
-  (segment (start 151.13 113.03) (end 152.4 111.76) (width 1.4) (layer F.Cu) (net 24))
-  (segment (start 152.4 111.76) (end 152.4 107.95) (width 1.4) (layer F.Cu) (net 24))
   (segment (start 156.23 104.14) (end 157.48 104.14) (width 0.25) (layer F.Cu) (net 24))
-  (segment (start 152.42 107.95) (end 156.23 104.14) (width 1.4) (layer F.Cu) (net 24))
-  (segment (start 152.4 107.95) (end 152.42 107.95) (width 0.25) (layer F.Cu) (net 24))
+  (segment (start 153.69 106.68) (end 156.23 104.14) (width 2.4) (layer F.Cu) (net 24))
+  (segment (start 153.67 106.68) (end 153.69 106.68) (width 0.25) (layer F.Cu) (net 24))
+  (segment (start 153.67 111.76) (end 153.67 106.68) (width 2.4) (layer F.Cu) (net 24))
+  (segment (start 152.4 113.03) (end 153.67 111.76) (width 2.4) (layer F.Cu) (net 24))
+  (segment (start 152.4 113.03) (end 149.86 113.03) (width 2.4) (layer F.Cu) (net 24))
+  (segment (start 149.86 82.55) (end 156.21 82.55) (width 0.25) (layer F.Cu) (net 26))
+  (segment (start 147.32 85.09) (end 149.86 82.55) (width 0.25) (layer F.Cu) (net 26))
+  (segment (start 142.24 85.09) (end 147.32 85.09) (width 0.25) (layer F.Cu) (net 26))
   (segment (start 129.54 86.36) (end 140.97 86.36) (width 0.25) (layer F.Cu) (net 26))
   (segment (start 140.97 86.36) (end 142.24 85.09) (width 0.25) (layer F.Cu) (net 26))
-  (segment (start 142.24 85.09) (end 146.05 85.09) (width 0.25) (layer F.Cu) (net 26))
-  (segment (start 148.59 82.55) (end 156.21 82.55) (width 0.25) (layer F.Cu) (net 26))
-  (segment (start 146.05 85.09) (end 148.59 82.55) (width 0.25) (layer F.Cu) (net 26))
   (segment (start 129.54 88.9) (end 140.97 88.9) (width 0.25) (layer F.Cu) (net 27))
   (segment (start 140.97 88.9) (end 142.24 87.63) (width 0.25) (layer F.Cu) (net 27))
