File: stairway-to-heaven-pcb/stairway-to-heaven-pcb.kicad_sch (KiCad schematic)
At the start: 8 parts, among them J15 PJ-063AH, J16 Conn_01x06_Male, U1 MEGA_PRO_EMBED_CH340G_{slash}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

Commit message: Organize footprints and symbols
Parts:
- J15: footprint kicad-ss-libs:CUI_PJ-063AH -> CUI_PJ-063AH
- RV100k1: footprint CA6V Potentiometer THT:CA6V-NoMidHole -> CA6V:CA6V-NoMidHole
- U1: footprint kicad:MEGA_PRO_EMBED_CH340G___ATMEGA2560 -> Mega2560MiniPro:MODULE_MEGA_PRO_EMBED_CH340G___ATMEGA2560
